File: PCB/Faikout/Faikout.kicad_pcb (KiCad board)
At the start: 2 copper layers, 70 x 70 mm, 47 parts, among them J1 1x5, J2 TC2030-USB-NL, J3 Reset, Q1 BSS138PS, U1 TPS562246, U4 ESP32-S3-MINI-1

Commit message: KiCAD 10
Parts:
- U4: value ESP32-S3-MINI-1 -> ESP32-S3-MINI-1-N4R2
Routing:
- net Net-(J3-Pin_2): track 7.10 -> 6.56 mm
